File: src/pcb/kicad/saw_carrier.kicad_sch (KiCad schematic)
At the start: 18 parts, among them J1 Conn_Coaxial, J2 Conn_Coaxial, U1 SAW_Sensor

Commit message: remove obsolete folder
Parts:
- added G1: logo, saw_sensor:hs_wismar_logo_12mmx9_2mm, symbol saw_sensor:logo
- added G2: logo, saw_sensor:hs_wismar_logo_6_2mmx5mm, symbol saw_sensor:logo
- H1, H2, H3, H4: footprint MountingHole:MountingHole_2.5mm -> MountingHole:MountingHole_3.2mm_M3
- renumbered C5 to C1, C6 to C2, C7 to C3, C1 to X1, C10 to X10, C11 to X11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
Other:
- moved on the sheet: H1, H2, X1
